File: drone.sch (KiCad schematic (older format))
At the start: 1 part

Commit message: Worked on the schematic somemore
Parts:
- added M1: Motor, symbol Motor
- added M2: StepperMotor, symbol StepperMotor
- added Q1, Q2: NPN, symbol NPN
- added U1: Relay_SPDT, symbol Relay_SPDT
- gave numbers to parts that had none: 1
Connections:
- net +12V: now also U1.~
- net GND: now reaches U2.~
- net GND: now also U1.~
- new net: M1.~, U2.~
- new net: Q1.1 (E), U2.~
- new net: Q2.1 (E), U1.~
- new net: M1.~, U1.~
- new net +5V: Q1.3 (C), Q2.3 (C)
Other:
- moved on the sheet: U2
Changed lines of the file:
@@
 LIBS:contrib
 LIBS:valves
+LIBS:drone-cache
 EELAYER 24 0
 EELAYER END
@@
 $EndDescr
 $Comp
-L +12V #PWR?
+L +12V #PWR5
 U 1 1 556A3819
-P 2450 1550
-F 0 "#PWR?" H 2450 1500 20  0001 C CNN
-F 1 "+12V" H 2450 1650 30  0000 C CNN
-F 2 "" H 2450 1550 60  0000 C CNN
-F 3 "" H 2450 1550 60  0000 C CNN
-	1    2450 1550
+P 2975 1725
+F 0 "#PWR5" H 2975 1675 20  0001 C CNN
+F 1 "+12V" H 2975 1825 30  0000 C CNN
+F 2 "" H 2975 1725 60  0000 C CNN
+F 3 "" H 2975 1725 60  0000 C CNN
+	1    2975 1725
 	1    0    0    -1
 $EndComp
 $Comp
-L Relay_SPDT U?
+L Relay_SPDT U2
 U 1 1 556A385C
-P 3300 2400
-F 0 "U?" H 3325 2250 60  0000 C CNN
-F 1 "Relay_SPDT" H 3325 2500 60  0000 C CNN
-F 2 "" H 3300 2400 60  0000 C CNN
-F 3 "" H 3300 2400 60  0000 C CNN
-	1    3300 2400
+P 2950 3300
+F 0 "U2" H 2975 3150 60  0000 C CNN
+F 1 "Relay_SPDT" H 2975 3400 60  0000 C CNN
+F 2 "" H 2950 3300 60  0000 C CNN
+F 3 "" H 2950 3300 60  0000 C CNN
+	1    2950 3300
+	0    1    1    0
+$EndComp
+$Comp
+L GND #PWR6
+U 1 1 556A391F
+P 3100 1850
+F 0 "#PWR6" H 3100 1850 30  0001 C CNN
+F 1 "GND" H 3100 1780 30  0001 C CNN
+F 2 "" H 3100 1850 60  0000 C CNN
+F 3 "" H 3100 1850 60  0000 C CNN
+	1    3100 1850
+	0    -1   -1   0
+$EndComp
+Wire Wire Line
+	3000 1950 3000 1850
+Wire Wire Line
+	3000 1850 3100 1850
+$Comp
+L NPN Q2
+U 1 1 556A39D3
+P 2700 1500
+F 0 "Q2" H 2700 1350 50  0000 R CNN
+F 1 "NPN" H 2700 1650 50  0000 R CNN
+F 2 "" H 2700 1500 60  0000 C CNN
+F 3 "" H 2700 1500 60  0000 C CNN
+	1    2700 1500
 	1    0    0    -1
 $EndComp
+Wire Wire Line
+	2800 1700 2800 1850
+Wire Wire Line
+	2800 1850 2850 1850
+$Comp
+L GND #PWR3
+U 1 1 556A39F6
+P 2850 2400
+F 0 "#PWR3" H 2850 2400 30  0001 C CNN
+F 1 "GND" H 2850 2330 30  0001 C CNN
+F 2 "" H 2850 2400 60  0000 C CNN
+F 3 "" H 2850 2400 60  0000 C CNN
+	1    2850 2400
+	1    0    0    -1
+$EndComp
+Wire Wire Line
+	2850 2400 2850 2350
+$Comp
+L GND #PWR4
+U 1 1 556A3A11
+P 2850 3600
+F 0 "#PWR4" H 2850 3600 30  0001 C CNN
+F 1 "GND" H 2850 3530 30  0001 C CNN
+F 2 "" H 2850 3600 60  0000 C CNN
+F 3 "" H 2850 3600 60  0000 C CNN
+	1    2850 3600
+	1    0    0    -1
+$EndComp
+Wire Wire Line
+	2850 3600 2850 3550
+$Comp
+L Motor M1
+U 1 1 556A3AEA
+P 2950 2700
+F 0 "M1" H 2950 2700 60  0000 C CNN
+F 1 "Motor" V 3075 2700 60  0000 C CNN
+F 2 "" H 2950 2700 60  0000 C CNN
+F 3 "" H 2950 2700 60  0000 C CNN
+	1    2950 2700
+	1    0    0    -1
+$EndComp
+Wire Wire Line
+	2950 3075 2950 3125
+Wire Wire Line
+	2950 2275 2950 2325
+$Comp
+L Relay_SPDT U1
+U 1 1 556A38E1
+P 2950 2100
+F 0 "U1" H 2975 1950 60  0000 C CNN
+F 1 "Relay_SPDT" H 2975 2200 60  0000 C CNN
+F 2 "" H 2950 2100 60  0000 C CNN
+F 3 "" H 2950 2100 60  0000 C CNN
+	1    2950 2100
+	0    1    -1   0
+$EndComp
+Wire Wire Line
+	2900 1950 2900 1725
+Wire Wire Line
+	2900 1725 2975 1725
+$Comp
+L +5V #PWR2
+U 1 1 556A3BDA
+P 2800 1250
+F 0 "#PWR2" H 2800 1340 20  0001 C CNN
+F 1 "+5V" H 2800 1340 30  0000 C CNN
+F 2 "" H 2800 1250 60  0000 C CNN
+F 3 "" H 2800 1250 60  0000 C CNN
+	1    2800 1250
+	1    0    0    -1
+$EndComp
+Wire Wire Line
+	2800 1300 2800 1250
+$Comp
+L NPN Q1
+U 1 1 556A3BFA
+P 2625 2750
+F 0 "Q1" H 2625 2600 50  0000 R CNN
+F 1 "NPN" H 2625 2900 50  0000 R CNN
+F 2 "" H 2625 2750 60  0000 C CNN
+F 3 "" H 2625 2750 60  0000 C CNN
+	1    2625 2750
+	1    0    0    -1
+$EndComp
+Wire Wire Line
+	2725 2950 2725 3050
+Wire Wire Line
+	2725 3050 2850 3050
+$Comp
+L +5V #PWR1
+U 1 1 556A3C22
+P 2725 2500
+F 0 "#PWR1" H 2725 2590 20  0001 C CNN
+F 1 "+5V" H 2725 2590 30  0000 C CNN
+F 2 "" H 2725 2500 60  0000 C CNN
+F 3 "" H 2725 2500 60  0000 C CNN
+	1    2725 2500
+	1    0    0    -1
+$EndComp
+Wire Wire Line
+	2725 2550 2725 2500
+$Comp
+L StepperMotor M2
+U 1 1 556A3F5C
+P 7500 4700
+F 0 "M2" H 7500 4500 60  0000 C CNN
+F 1 "StepperMotor" H 7525 4925 60  0000 C CNN
+F 2 "" H 7525 4700 60  0000 C CNN
+F 3 "" H 7525 4700 60  0000 C CNN
+	1    7500 4700
+	1    0    0    -1
+$EndComp
